Commit message: removed dummy object collision and changed table color

File: SwapWith-Universal_Robot/ur_description/urdf/inc/ur_macro.xacro (robot description, xacro)
@@ -384,5 +384,7 @@
 				<box size=".7 1 .1"/>
 			</geometry>
-			<material name="LightGrey"/>
+			<material name="DarkGrey">
+				<color rgba="0.0 0.0 0.0.0.8"/>
+			</material>
 		</visual>
 		<collision>
@@ -406,17 +408,10 @@
   		</material>
 		</visual>
-		<collision>
-			<geometry>
-				<box size="0.01 0.6 0.01"/>
-			</geometry>
-		</collision>
-		<inertial>
-      <mass value="1e-5" />
-      <origin xyz="0 0 0" rpy="0 0 0"/>
-      <inertia ixx="1e-6" ixy="0" ixz="0" iyy="1e-6" iyz="0" izz="1e-6" />
-    </inertial>
 	</link>
 	<gazebo reference="dummy_link">
   <material>Gazebo/Blue</material>
+  </gazebo>
+  <gazebo reference="table_link">
+  <material>Gazebo/DarkGrey</material>
   </gazebo>
 	<joint name="ground_joint" type="fixed">

Commit message: updated project to mimic irl setup. Need to adjust haptic values for manipulaitng the robot. Reaches edge before contact with target.

File: SwapWith-Universal_Robot/ur_description/urdf/inc/ur_macro.xacro (robot description, xacro)
@@ -343,16 +343,13 @@
       <child link="${prefix}tool0"/>
     </joint>
-  <link name="ground_link">
-    <visual>
-			<geometry>
-				<box size="10 10 .01"/>
-			</geometry>
-			<material name="LightGrey"/>
+  <link name="checkerboard_link">
+    <visual>
+			<geometry>
+				<box size=".085 .085 .01"/>
+			</geometry>
+			<material name="Black">
+   			<color rgba="0.0 0.0 0.0 1.0"/>
+  		</material>
 		</visual>
-		<collision>
-			<geometry>
-				<box size="10 10 .01"/>
-			</geometry>
-		</collision>
 		<inertial>
       <mass value="1e-5" />
@@ -361,36 +358,14 @@
     </inertial>
 	</link>
-	<link name="wall_link1">
-    <visual>
-			<geometry>
-				<box size="3 0 3"/>
+	<gazebo reference="checkerboard_link">
+  <material>Gazebo/Black</material>
+  </gazebo>
+  <link name="table_link">
+    <visual>
+			<geometry>
+				<box size=".5 .5 .01"/>
 			</geometry>
 			<material name="LightGrey"/>
 		</visual>
-		<collision>
-			<geometry>
-				<box size="3 0 3"/>
-			</geometry>
-		</collision>
-		<inertial>
-      <mass value="1e-5" />
-      <origin xyz="0 0 0" rpy="0 0 0"/>
-      <inertia ixx="1e-6" ixy="0" ixz="0" iyy="1e-6" iyz="0" izz="1e-6" />
-    </inertial>
-	</link>
-  <link name="table_link">
-    <visual>
-			<geometry>
-				<box size=".7 1 .1"/>
-			</geometry>
-			<material name="DarkGrey">
-				<color rgba="0.0 0.0 0.0.0.8"/>
-			</material>
-		</visual>
-		<collision>
-			<geometry>
-				<box size=".7 1 .1"/>
-			</geometry>
-		</collision>
 		<inertial>
       <mass value="1e-5" />
@@ -402,5 +377,5 @@
     <visual>
 			<geometry>
-				<box size="0.01 0.6 0.01"/>
+				<box size="0.01 0.3 0.01"/>
 			</geometry>
 			<material name="Blue">
@@ -408,43 +383,39 @@
   		</material>
 		</visual>
+		<collision>
+			<geometry>
+				<box size="0.01 0.3 0.01"/>
+			</geometry>
+		</collision>
+		<inertial>
+      <mass value="1e-5" />
+      <origin xyz="0 0 0" rpy="0 0 0"/>
+      <inertia ixx="1e-6" ixy="0" ixz="0" iyy="1e-6" iyz="0" izz="1e-6" />
+    </inertial>
 	</link>
 	<gazebo reference="dummy_link">
   <material>Gazebo/Blue</material>
   </gazebo>
-  <gazebo reference="table_link">
-  <material>Gazebo/DarkGrey</material>
-  </gazebo>
-	<joint name="ground_joint" type="fixed">
-      <parent link="world" />
-      <child link="ground_link" />
-      <origin xyz="0 -0.1 0" rpy="0 0 0" />
-    </joint>
-  <joint name="wall_joint1" type="fixed">
-      <parent link="world" />
-      <child link="wall_link1" />
-      <origin xyz="1 0 0" rpy="0 0 1.57" />
+	<joint name="checkered_joint" type="fixed">
+      <parent link="base" />
+      <child link="checkerboard_link" />
+      <origin xyz="0.00937 -0.4906 0" rpy="0 0 -1.5708" />
     </joint>
 	<joint name="table_joint" type="fixed">
-      <parent link="world" />
+      <parent link="checkerboard_link" />
       <child link="table_link" />
-      <origin xyz="-0.5 0 0" rpy="0 0 0" />
+      <origin xyz="0.3 -0.1 .01" rpy="0 0 0" />
     </joint>
   <joint name="dummy_joint" type="fixed">
       <parent link="table_link" />
       <child link="dummy_link" />
-      <origin xyz="0 0 .1" rpy="0 -1.57 0" />
+      <origin xyz="0 0 .05" rpy="0 -1.57 0" />
     </joint>
     <!-- Camera left -->
   <link name="left_camera_link">
-    <collision>
+    <visual>
       <origin xyz="0 0 0" rpy="0 0 0"/>
       <geometry>
-    <box size=".05 .05 .05"/>
-      </geometry>
-    </collision>
-    <visual>
-      <origin xyz="0 0 0" rpy="0 0 0"/>
-      <geometry>
-    <box size=".05 .05 .05"/>
+    <box size=".02 .02 .02"/>
       </geometry>
       <material name="LightGrey"/>
@@ -457,8 +428,7 @@
   </link>
   <joint name="left_camera_joint" type="fixed">
-      <parent link="world" />
+      <parent link="checkerboard_link" />
       <child link="left_camera_link" />
-      <!-- change y of rpy to rotate x around (if -y in xyz, use + y in rpy) -->
-      <origin xyz="-1.2 0.05 .6" rpy="0 0.7 0" />
+      <origin xyz="0.372 -0.041 0.362" rpy="0.680144 1.43376 -2.9968" />
     </joint>
     <!-- generate an optical frame http://www.ros.org/reps/rep-0103.html#suffix-frames
@@ -477,14 +447,8 @@
   <!-- Camera -->
   <link name="right_camera_link">
-    <collision>
+    <visual>
       <origin xyz="0 0 0" rpy="0 0 0"/>
       <geometry>
-    <box size=".05 .05 .05"/>
-      </geometry>
-    </collision>
-    <visual>
-      <origin xyz="0 0 0" rpy="0 0 0"/>
-      <geometry>
-    <box size=".05 .05 .05"/>
+    <box size=".02 .02 .02"/>
       </geometry>
       <material name="LightGrey"/>
@@ -496,9 +460,47 @@
     </inertial>
   </link>
+  <link name="middle_camera_link">
+    <visual>
+      <origin xyz="0 0 0" rpy="0 0 0"/>
+      <geometry>
+    <box size=".02 .02 .02"/>
+      </geometry>
+      <material name="LightGrey"/>
+    </visual>
+    <inertial>
+      <mass value="1e-5" />
+      <origin xyz="0 0 0" rpy="0 0 0"/>
+      <inertia ixx="1e-6" ixy="0" ixz="0" iyy="1e-6" iyz="0" izz="1e-6" />
+    </inertial>
+  </link>
+  <link name="intel_camera_link">
+    <visual>
+      <origin xyz="0 0 0" rpy="0 0 0"/>
+      <geometry>
+    <box size=".02 .02 .02"/>
+      </geometry>
+      <material name="LightGrey"/>
+    </visual>
+    <inertial>
+      <mass value="1e-5" />
+      <origin xyz="0 0 0" rpy="0 0 0"/>
+      <inertia ixx="1e-6" ixy="0" ixz="0" iyy="1e-6" iyz="0" izz="1e-6" />
+    </inertial>
+  </link>
   <joint name="right_camera_joint" type="fixed">
-      <parent link="left_camera_link" />
+      <parent link="checkerboard_link" />
       <child link="right_camera_link" />
-      <!-- change y of rpy to rotate x around (if -y in xyz, use + y in rpy) -->
-      <origin xyz="0 -0.1 0" rpy="0 0 0" />
+      <origin xyz="0.358 0.032 0.374" rpy="0.58108 1.2832755 -2.7483" />
+    </joint>
+    <!-- -2.7483 -0.58108 -1.2832755 -->
+  <joint name="middle_camera_joint" type="fixed">
+      <parent link="checkerboard_link" />
+      <child link="middle_camera_link" />
+      <origin xyz="0.365 -0.0045 0.368" rpy="0.630597 1.35851775 -2.87255" />
+    </joint>
+  <joint name="intel_camera_joint" type="fixed">
+      <parent link="checkerboard_link" />
+      <child link="intel_camera_link" />
+      <origin xyz="0.316 -0.177 0.327" rpy="0.673 1.4905 -3.0835" />
     </joint>
     <!-- generate an optical frame http://www.ros.org/reps/rep-0103.html#suffix-frames
@@ -514,4 +516,11 @@
   </joint>
   <link name="camera_link_optical_right">
+  </link>
+  <joint name="middle_camera_optical_joint" type="fixed">
+    <origin xyz="0 0 0" rpy="-1.57079632679 0 -1.57079632679"/>
+    <parent link="middle_camera_link"/>
+    <child link="camera_link_optical_middle"/>
+  </joint>
+  <link name="camera_link_optical_middle">
   </link>
   <xacro:property name="link_name1" value="left_camera_link" />
@@ -599,4 +608,86 @@
     </sensor>
   </gazebo>
+  <!-- camera middle -->
+	 <gazebo reference="middle_camera_link">
+    <sensor type="camera" name="virtual_camera_middle">
+      <update_rate>30.0</update_rate>
+      <camera name="middle">
+        <horizontal_fov>1.3962634</horizontal_fov>
+        <image>
+          <width>800</width>
+          <height>800</height>
+          <format>R8G8B8</format>
+        </image>
+        <clip>
+          <near>0.02</near>
+          <far>300</far>
+        </clip>
+        <noise>
+          <type>gaussian</type>
+          <!-- Noise is sampled independently per pixel on each frame.
+               That pixel's noise value is added to each of its color
+               channels, which at that point lie in the range [0,1]. -->
+          <mean>0.0</mean>
+          <stddev>0.007</stddev>
+        </noise>
+      </camera>
+      <plugin name="camera_controller" filename="libgazebo_ros_camera.so">
+        <alwaysOn>true</alwaysOn>
+        <updateRate>0.0</updateRate>
+        <cameraName>middle</cameraName>
+        <imageTopicName>image_raw</imageTopicName>
+        <cameraInfoTopicName>camera_info</cameraInfoTopicName>
+        <frameName>camera_link_optical_middle</frameName>
+        <hackBaseline>0.07</hackBaseline>
+        <distortionK1>0.0</distortionK1>
+        <distortionK2>0.0</distortionK2>
+        <distortionK3>0.0</distortionK3>
+        <distortionT1>0.0</distortionT1>
+        <distortionT2>0.0</distortionT2>
+      </plugin>
+    </sensor>
+  </gazebo>
+  <!-- camera intel -->
+  <gazebo reference="intel_camera_link">
+		<sensor name="intel_camera" type="depth">
+		  <update_rate>20</update_rate>
+		  <camera>
+		    <horizontal_fov>1.047198</horizontal_fov>
+		    <image>
+		      <width>640</width>
+		      <height>480</height>
+		      <format>R8G8B8</format>
+		    </image>
+		    <clip>
+		      <near>0.05</near>
+		      <far>3</far>
+		    </clip>
+		  </camera>
+		  <plugin name="intel_camera_link_controller" filename="libgazebo_ros_openni_kinect.so">
+		    <baseline>0.2</baseline>
+		    <alwaysOn>true</alwaysOn>
+		    <updateRate>1.0</updateRate>
+		    <cameraName>intel_ir</cameraName>
+		    <imageTopicName>/intel/color/image_raw</imageTopicName>
+		    <cameraInfoTopicName>/intel/color/camera_info</cameraInfoTopicName>
+		    <depthImageTopicName>/inteldepth/image_raw</depthImageTopicName>
+		    <depthImageInfoTopicName>/intel/depth/camera_info</depthImageInfoTopicName>
+		    <pointCloudTopicName>/intel/depth/points</pointCloudTopicName>
+		    <frameName>intel_frame</frameName>
+		    <pointCloudCutoff>0.5</pointCloudCutoff>
+		    <pointCloudCutoffMax>3.0</pointCloudCutoffMax>
+		    <distortionK1>0.00000001</distortionK1>
+		    <distortionK2>0.00000001</distortionK2>
+		    <distortionK3>0.00000001</distortionK3>
+		    <distortionT1>0.00000001</distortionT1>
+		    <distortionT2>0.00000001</distortionT2>
+		    <CxPrime>0</CxPrime>
+		    <Cx>0</Cx>
+		    <Cy>0</Cy>
+		    <focalLength>0</focalLength>
+		    <hackBaseline>0</hackBaseline>
+		  </plugin>
+		</sensor>
+	</gazebo>
   </xacro:macro>
 </robot>

Commit message: Overlay will show somethign, but not correct.

File: SwapWith-Universal_Robot/ur_description/urdf/inc/ur_macro.xacro (robot description, xacro)
@@ -383,9 +383,4 @@
   		</material>
 		</visual>
-		<collision>
-			<geometry>
-				<box size="0.01 0.3 0.01"/>
-			</geometry>
-		</collision>
 		<inertial>
       <mass value="1e-5" />
@@ -674,5 +669,5 @@
 		    <depthImageInfoTopicName>/intel/depth/camera_info</depthImageInfoTopicName>
 		    <pointCloudTopicName>/intel/depth/points</pointCloudTopicName>
-		    <frameName>intel_frame</frameName>
+		    <frameName>intel_camera_link</frameName>
 		    <pointCloudCutoff>0.5</pointCloudCutoff>
 		    <pointCloudCutoffMax>3.0</pointCloudCutoffMax>

Commit message: Added launch parameters to plan_listener and listener. Updated simulation cameras to reflect real world. Need to update table and test sample.

File: SwapWith-Universal_Robot/ur_description/urdf/inc/ur_macro.xacro (robot description, xacro)
@@ -395,5 +395,5 @@
       <parent link="base" />
       <child link="checkerboard_link" />
-      <origin xyz="0.00937 -0.4906 0" rpy="0 0 -1.5708" />
+      <origin xyz="-0.06496 -0.47047 0.001" rpy="0 0 -1.5708" />
     </joint>
 	<joint name="table_joint" type="fixed">
@@ -424,7 +424,9 @@
   <joint name="left_camera_joint" type="fixed">
       <parent link="checkerboard_link" />
-      <child link="left_camera_link" />
-      <origin xyz="0.372 -0.041 0.362" rpy="0.680144 1.43376 -2.9968" />
-    </joint>
+      <child link="camera_link_optical_left" />
+      <origin xyz="0.447 0.019 0.440" rpy="-2.367 -0.025 1.507" />
+    </joint>
+   <link name="camera_link_optical_left">
+  </link>
     <!-- generate an optical frame http://www.ros.org/reps/rep-0103.html#suffix-frames
       so that ros and opencv can operate on the camera frame correctly -->
@@ -434,10 +436,8 @@
     <!-- Make sure the frame name is set to the optical one under the camera sensor
     	  settings. The optical link is for depth camera specifically -->
-    <origin xyz="0 0 0" rpy="-1.57079632679 0 -1.57079632679"/>
-    <parent link="left_camera_link"/>
-    <child link="camera_link_optical_left"/>
+    <origin xyz="0 0 0" rpy="1.57079632679 -1.57079632679 0"/>
+    <parent link="camera_link_optical_left"/>
+    <child link="left_camera_link"/>
   </joint>
-  <link name="camera_link_optical_left">
-  </link>
   <!-- Camera -->
   <link name="right_camera_link">
@@ -455,5 +455,5 @@
     </inertial>
   </link>
-  <link name="middle_camera_link">
+  <link name="intel_camera_link">
     <visual>
       <origin xyz="0 0 0" rpy="0 0 0"/>
@@ -469,29 +469,10 @@
     </inertial>
   </link>
-  <link name="intel_camera_link">
-    <visual>
-      <origin xyz="0 0 0" rpy="0 0 0"/>
-      <geometry>
-    <box size=".02 .02 .02"/>
-      </geometry>
-      <material name="LightGrey"/>
-    </visual>
-    <inertial>
-      <mass value="1e-5" />
-      <origin xyz="0 0 0" rpy="0 0 0"/>
-      <inertia ixx="1e-6" ixy="0" ixz="0" iyy="1e-6" iyz="0" izz="1e-6" />
-    </inertial>
-  </link>
   <joint name="right_camera_joint" type="fixed">
       <parent link="checkerboard_link" />
-      <child link="right_camera_link" />
-      <origin xyz="0.358 0.032 0.374" rpy="0.58108 1.2832755 -2.7483" />
+      <child link="camera_link_optical_right" />
+      <origin xyz="0.450 0.095 0.437" rpy="-2.363 0.052 1.568" />
     </joint>
     <!-- -2.7483 -0.58108 -1.2832755 -->
-  <joint name="middle_camera_joint" type="fixed">
-      <parent link="checkerboard_link" />
-      <child link="middle_camera_link" />
-      <origin xyz="0.365 -0.0045 0.368" rpy="0.630597 1.35851775 -2.87255" />
-    </joint>
   <joint name="intel_camera_joint" type="fixed">
       <parent link="checkerboard_link" />
@@ -506,16 +487,9 @@
     <!-- Make sure the frame name is set to the optical one under the camera sensor
     	  settings. The optical link is for depth camera specifically -->
-    <origin xyz="0 0 0" rpy="-1.57079632679 0 -1.57079632679"/>
-    <parent link="right_camera_link"/>
-    <child link="camera_link_optical_right"/>
+    <origin xyz="0 0 0" rpy="1.57079632679 -1.57079632679 0"/>
+    <parent link="camera_link_optical_right"/>
+    <child link="right_camera_link"/>
   </joint>
   <link name="camera_link_optical_right">
-  </link>
-  <joint name="middle_camera_optical_joint" type="fixed">
-    <origin xyz="0 0 0" rpy="-1.57079632679 0 -1.57079632679"/>
-    <parent link="middle_camera_link"/>
-    <child link="camera_link_optical_middle"/>
-  </joint>
-  <link name="camera_link_optical_middle">
   </link>
   <xacro:property name="link_name1" value="left_camera_link" />
@@ -603,44 +577,4 @@
     </sensor>
   </gazebo>
-  <!-- camera middle -->
-	 <gazebo reference="middle_camera_link">
-    <sensor type="camera" name="virtual_camera_middle">
-      <update_rate>30.0</update_rate>
-      <camera name="middle">
-        <horizontal_fov>1.3962634</horizontal_fov>
-        <image>
-          <width>800</width>
-          <height>800</height>
-          <format>R8G8B8</format>
-        </image>
-        <clip>
-          <near>0.02</near>
-          <far>300</far>
-        </clip>
-        <noise>
-          <type>gaussian</type>
-          <!-- Noise is sampled independently per pixel on each frame.
-               That pixel's noise value is added to each of its color
-               channels, which at that point lie in the range [0,1]. -->
-          <mean>0.0</mean>
-          <stddev>0.007</stddev>
-        </noise>
-      </camera>
-      <plugin name="camera_controller" filename="libgazebo_ros_camera.so">
-        <alwaysOn>true</alwaysOn>
-        <updateRate>0.0</updateRate>
-        <cameraName>middle</cameraName>
-        <imageTopicName>image_raw</imageTopicName>
-        <cameraInfoTopicName>camera_info</cameraInfoTopicName>
-        <frameName>camera_link_optical_middle</frameName>
-        <hackBaseline>0.07</hackBaseline>
-        <distortionK1>0.0</distortionK1>
-        <distortionK2>0.0</distortionK2>
-        <distortionK3>0.0</distortionK3>
-        <distortionT1>0.0</distortionT1>
-        <distortionT2>0.0</distortionT2>
-      </plugin>
-    </sensor>
-  </gazebo>
   <!-- camera intel -->
   <gazebo reference="intel_camera_link">

Commit message: fixed haptic force during teleoperation. Changed simulation models. Added simple data logger

File: SwapWith-Universal_Robot/ur_description/urdf/inc/ur_macro.xacro (robot description, xacro)
@@ -308,5 +308,5 @@
     <visual>
 			<geometry>
-				<cylinder length="0.06" radius="0.02"/>
+				<cylinder length="0.01" radius="0.03"/>
 			</geometry>
 			<material name="LightGrey"/>
@@ -314,5 +314,5 @@
 		<collision>
 			<geometry>
-				<cylinder length="0.06" radius="0.02"/>
+				<cylinder length="0.01" radius="0.03"/>
 			</geometry>
 		</collision>
@@ -321,5 +321,5 @@
       <parent link="${prefix}wrist_3_link" />
       <child link="${prefix}flange" />
-      <origin xyz="0 0 .03" rpy="0 0 0" />
+      <origin xyz="0 0 .005" rpy="0 0 0" />
     </joint>
     <!-- ROS-Industrial 'tool0' frame: all-zeros tool frame -->
@@ -327,5 +327,5 @@
 		<visual>
 			<geometry>
-				<cylinder length="0.06" radius="0.005"/>
+				<cylinder length="0.12" radius="0.01"/>
 			</geometry>
 			<material name="LightGrey"/>
@@ -333,8 +333,23 @@
 		<collision>
 			<geometry>
-				<cylinder length="0.06" radius="0.005"/>
+				<cylinder length="0.12" radius="0.01"/>
 			</geometry>
 		</collision>
 	</link>
+	<link name="${prefix}needle">
+		<visual>
+			<geometry>
+				<cylinder length="0.0285" radius="0.001"/>
+			</geometry>
+		</visual>
+		<collision>
+			<geometry>
+				<cylinder length="0.0285" radius="0.001"/>
+			</geometry>
+		</collision>
+	</link>
+	<gazebo reference="${prefix}needle">
+  <material>Gazebo/Black</material>
+  </gazebo>
     <joint name="${prefix}flange-tool0" type="fixed">
       <!-- default toolframe: X+ left, Y+ up, Z+ front -->
@@ -343,4 +358,10 @@
       <child link="${prefix}tool0"/>
     </joint>
+    <joint name="${prefix}tool0-needle" type="fixed">
+      <!-- default toolframe: X+ left, Y+ up, Z+ front -->
+      <origin xyz="0 0 0.07425" rpy="0 0 0"/>
+      <parent link="${prefix}tool0"/>
+      <child link="${prefix}needle"/>
+    </joint>
   <link name="checkerboard_link">
     <visual>
@@ -348,7 +369,4 @@
 				<box size=".085 .085 .01"/>
 			</geometry>
-			<material name="Black">
-   			<color rgba="0.0 0.0 0.0 1.0"/>
-  		</material>
 		</visual>
 		<inertial>
@@ -374,12 +392,9 @@
     </inertial>
 	</link>
-	<link name="dummy_link">
-    <visual>
-			<geometry>
-				<box size="0.01 0.3 0.01"/>
-			</geometry>
-			<material name="Blue">
-   			<color rgba="0.0 0.0 0.8 1.0"/>
-  		</material>
+	<link name="dummy_link_ns">
+    <visual>
+			<geometry>
+				<box size="0.01 0.3 0.03"/>
+			</geometry>
 		</visual>
 		<inertial>
@@ -389,5 +404,20 @@
     </inertial>
 	</link>
-	<gazebo reference="dummy_link">
+	<link name="dummy_link_ew">
+    <visual>
+			<geometry>
+				<box size="0.01 0.3 0.03"/>
+			</geometry>
+		</visual>
+		<inertial>
+      <mass value="1e-5" />
+      <origin xyz="0 0 0" rpy="0 0 0"/>
+      <inertia ixx="1e-6" ixy="0" ixz="0" iyy="1e-6" iyz="0" izz="1e-6" />
+    </inertial>
+	</link>
+	<gazebo reference="dummy_link_ns">
+  <material>Gazebo/Blue</material>
+  </gazebo>
+  <gazebo reference="dummy_link_ew">
   <material>Gazebo/Blue</material>
   </gazebo>
@@ -400,10 +430,22 @@
       <parent link="checkerboard_link" />
       <child link="table_link" />
-      <origin xyz="0.3 -0.1 .01" rpy="0 0 0" />
-    </joint>
-  <joint name="dummy_joint" type="fixed">
+      <origin xyz=".01 0.05 .01" rpy="0 0 0" />
+    </joint>
+  <joint name="dummy_ns_joint" type="fixed">
       <parent link="table_link" />
-      <child link="dummy_link" />
-      <origin xyz="0 0 .05" rpy="0 -1.57 0" />
+      <child link="dummy_link_ns" />
+      <origin xyz="0 0 .015" rpy="0 0 0" />
+    </joint>
+  <joint name="dummy_ew_joint" type="fixed">
+      <parent link="table_link" />
+      <child link="dummy_link_ew" />
+      <origin xyz="0 0 .015" rpy="0 0 -1.57" />
+    </joint>
+  <link name="camera_user">
+  </link>
+ 	<joint name="user_joint" type="fixed">
+      <parent link="checkerboard_link" />
+      <child link="camera_user" />
+      <origin xyz="0.4485 0.057 0.4385" rpy="-2.366 0.014 1.537" />
     </joint>
     <!-- Camera left -->
@@ -427,5 +469,12 @@
       <origin xyz="0.447 0.019 0.440" rpy="-2.367 -0.025 1.507" />
     </joint>
+   <joint name="left_camera_end_joint" type="fixed">
+      <parent link="camera_link_optical_left" />
+      <child link="camera_link_pos_left" />
+      <origin xyz="-0.07 0 0" rpy="0 0 0" />
+    </joint>
    <link name="camera_link_optical_left">
+  </link>
+  <link name="camera_link_pos_left">
   </link>
     <!-- generate an optical frame http://www.ros.org/reps/rep-0103.html#suffix-frames
@@ -491,5 +540,12 @@
     <child link="right_camera_link"/>
   </joint>
+  <joint name="right_camera_end_joint" type="fixed">
+      <parent link="camera_link_optical_right" />
+      <child link="camera_link_pos_right" />
+      <origin xyz="-0.07 0 0" rpy="0 0 0" />
+    </joint>
   <link name="camera_link_optical_right">
+  </link>
+  <link name="camera_link_pos_right">
   </link>
   <xacro:property name="link_name1" value="left_camera_link" />
@@ -527,5 +583,5 @@
         <imageTopicName>image_raw</imageTopicName>
         <cameraInfoTopicName>camera_info</cameraInfoTopicName>
-        <frameName>camera_link_optical_left</frameName>
+        <frameName>camera_link_pos_left</frameName>
         <hackBaseline>0.07</hackBaseline>
         <distortionK1>0.0</distortionK1>
@@ -567,5 +623,5 @@
         <imageTopicName>image_raw</imageTopicName>
         <cameraInfoTopicName>camera_info</cameraInfoTopicName>
-        <frameName>camera_link_optical_right</frameName>
+        <frameName>camera_link_pos_right</frameName>
         <hackBaseline>0.07</hackBaseline>
         <distortionK1>0.0</distortionK1>
