Commit message: simulation model is smaller and closer

File: SwapWith-Universal_Robot/ur_description/urdf/inc/ur_macro.xacro (robot description, xacro)
@@ -340,15 +340,15 @@
 		<visual>
 			<geometry>
-				<cylinder length="0.0285" radius="0.001"/>
+				<cylinder length="0.0285" radius="0.0005"/>
 			</geometry>
 		</visual>
 		<collision>
 			<geometry>
-				<cylinder length="0.0285" radius="0.001"/>
+				<cylinder length="0.0285" radius="0.0005"/>
 			</geometry>
 		</collision>
 	</link>
 	<gazebo reference="${prefix}needle">
-  <material>Gazebo/Black</material>
+  <material>Gazebo/Yellow</material>
   </gazebo>
     <joint name="${prefix}flange-tool0" type="fixed">
@@ -367,5 +367,5 @@
     <visual>
 			<geometry>
-				<box size=".085 .085 .01"/>
+				<box size=".085 .085 .001"/>
 			</geometry>
 		</visual>
@@ -377,5 +377,5 @@
 	</link>
 	<gazebo reference="checkerboard_link">
-  <material>Gazebo/Black</material>
+  <material>Gazebo/Green</material>
   </gazebo>
   <link name="table_link">
@@ -395,5 +395,5 @@
     <visual>
 			<geometry>
-				<box size="0.01 0.3 0.03"/>
+				<box size="0.002 0.03 0.005"/>
 			</geometry>
 		</visual>
@@ -407,5 +407,5 @@
     <visual>
 			<geometry>
-				<box size="0.01 0.3 0.03"/>
+				<box size="0.002 0.03 0.005"/>
 			</geometry>
 		</visual>
@@ -425,20 +425,20 @@
       <parent link="base" />
       <child link="checkerboard_link" />
-      <origin xyz="-0.06496 -0.47047 0.001" rpy="0 0 -1.5708" />
+      <origin xyz="-0.06496 -0.47047 0.005" rpy="0 0 -1.5708" />
     </joint>
 	<joint name="table_joint" type="fixed">
       <parent link="checkerboard_link" />
       <child link="table_link" />
-      <origin xyz=".01 0.05 .01" rpy="0 0 0" />
+      <origin xyz=".38 0.02 .001" rpy="0 0 0" />
     </joint>
   <joint name="dummy_ns_joint" type="fixed">
       <parent link="table_link" />
       <child link="dummy_link_ns" />
-      <origin xyz="0 0 .015" rpy="0 0 0" />
+      <origin xyz="0 0 .005" rpy="0 0 0" />
     </joint>
   <joint name="dummy_ew_joint" type="fixed">
       <parent link="table_link" />
       <child link="dummy_link_ew" />
-      <origin xyz="0 0 .015" rpy="0 0 -1.57" />
+      <origin xyz="0 0 .005" rpy="0 0 -1.57" />
     </joint>
   <link name="camera_user">
@@ -464,25 +464,9 @@
     </inertial>
   </link>
-  <joint name="left_camera_joint" type="fixed">
-      <parent link="checkerboard_link" />
-      <child link="camera_link_optical_left" />
-      <origin xyz="0.447 0.019 0.440" rpy="-2.367 -0.025 1.507" />
-    </joint>
-   <joint name="left_camera_end_joint" type="fixed">
-      <parent link="camera_link_optical_left" />
-      <child link="camera_link_pos_left" />
-      <origin xyz="-0.07 0 0" rpy="0 0 0" />
-    </joint>
    <link name="camera_link_optical_left">
   </link>
   <link name="camera_link_pos_left">
   </link>
-    <!-- generate an optical frame http://www.ros.org/reps/rep-0103.html#suffix-frames
-      so that ros and opencv can operate on the camera frame correctly -->
   <joint name="left_camera_optical_joint" type="fixed">
-    <!-- these values have to be these values otherwise the gazebo camera image
-        won't be aligned properly with the frame it is supposedly originating from -->
-    <!-- Make sure the frame name is set to the optical one under the camera sensor
-    	  settings. The optical link is for depth camera specifically -->
     <origin xyz="0 0 0" rpy="1.57079632679 -1.57079632679 0"/>
     <parent link="camera_link_optical_left"/>
@@ -504,36 +488,20 @@
     </inertial>
   </link>
-  <link name="intel_camera_link">
-    <visual>
-      <origin xyz="0 0 0" rpy="0 0 0"/>
-      <geometry>
-    <box size=".02 .02 .02"/>
-      </geometry>
-      <material name="LightGrey"/>
-    </visual>
-    <inertial>
-      <mass value="1e-5" />
-      <origin xyz="0 0 0" rpy="0 0 0"/>
-      <inertia ixx="1e-6" ixy="0" ixz="0" iyy="1e-6" iyz="0" izz="1e-6" />
-    </inertial>
-  </link>
+  <joint name="left_camera_joint" type="fixed">
+      <parent link="checkerboard_link" />
+      <child link="camera_link_optical_left" />
+      <origin xyz="0.447 0.019 0.090" rpy="-2.367 -0.025 1.507" />
+    </joint>
+   <joint name="left_camera_end_joint" type="fixed">
+      <parent link="camera_link_optical_left" />
+      <child link="camera_link_pos_left" />
+      <origin xyz="-0.07 0 0" rpy="0 0 0" />
+    </joint>
   <joint name="right_camera_joint" type="fixed">
       <parent link="checkerboard_link" />
       <child link="camera_link_optical_right" />
-      <origin xyz="0.450 0.095 0.437" rpy="-2.363 0.052 1.568" />
-    </joint>
-    <!-- -2.7483 -0.58108 -1.2832755 -->
-  <joint name="intel_camera_joint" type="fixed">
-      <parent link="checkerboard_link" />
-      <child link="intel_camera_link" />
-      <origin xyz="0.316 -0.177 0.327" rpy="0.673 1.4905 -3.0835" />
-    </joint>
-    <!-- generate an optical frame http://www.ros.org/reps/rep-0103.html#suffix-frames
-      so that ros and opencv can operate on the camera frame correctly -->
+      <origin xyz="0.450 0.0325 0.090" rpy="-2.363 0.052 1.568" />
+    </joint>
   <joint name="right_camera_optical_joint" type="fixed">
-    <!-- these values have to be these values otherwise the gazebo camera image
-        won't be aligned properly with the frame it is supposedly originating from -->
-    <!-- Make sure the frame name is set to the optical one under the camera sensor
-    	  settings. The optical link is for depth camera specifically -->
     <origin xyz="0 0 0" rpy="1.57079632679 -1.57079632679 0"/>
     <parent link="camera_link_optical_right"/>
@@ -560,6 +528,6 @@
         <horizontal_fov>1.3962634</horizontal_fov>
         <image>
-          <width>800</width>
-          <height>800</height>
+          <width>1400</width>
+          <height>1400</height>
           <format>R8G8B8</format>
         </image>
@@ -600,6 +568,6 @@
         <horizontal_fov>1.3962634</horizontal_fov>
         <image>
-          <width>800</width>
-          <height>800</height>
+          <width>1400</width>
+          <height>1400</height>
           <format>R8G8B8</format>
         </image>
@@ -633,46 +601,4 @@
     </sensor>
   </gazebo>
-  <!-- camera intel -->
-  <gazebo reference="intel_camera_link">
-		<sensor name="intel_camera" type="depth">
-		  <update_rate>20</update_rate>
-		  <camera>
-		    <horizontal_fov>1.047198</horizontal_fov>
-		    <image>
-		      <width>640</width>
-		      <height>480</height>
-		      <format>R8G8B8</format>
-		    </image>
-		    <clip>
-		      <near>0.05</near>
-		      <far>3</far>
-		    </clip>
-		  </camera>
-		  <plugin name="intel_camera_link_controller" filename="libgazebo_ros_openni_kinect.so">
-		    <baseline>0.2</baseline>
-		    <alwaysOn>true</alwaysOn>
-		    <updateRate>1.0</updateRate>
-		    <cameraName>intel_ir</cameraName>
-		    <imageTopicName>/intel/color/image_raw</imageTopicName>
-		    <cameraInfoTopicName>/intel/color/camera_info</cameraInfoTopicName>
-		    <depthImageTopicName>/inteldepth/image_raw</depthImageTopicName>
-		    <depthImageInfoTopicName>/intel/depth/camera_info</depthImageInfoTopicName>
-		    <pointCloudTopicName>/intel/depth/points</pointCloudTopicName>
-		    <frameName>intel_camera_link</frameName>
-		    <pointCloudCutoff>0.5</pointCloudCutoff>
-		    <pointCloudCutoffMax>3.0</pointCloudCutoffMax>
-		    <distortionK1>0.00000001</distortionK1>
-		    <distortionK2>0.00000001</distortionK2>
-		    <distortionK3>0.00000001</distortionK3>
-		    <distortionT1>0.00000001</distortionT1>
-		    <distortionT2>0.00000001</distortionT2>
-		    <CxPrime>0</CxPrime>
-		    <Cx>0</Cx>
-		    <Cy>0</Cy>
-		    <focalLength>0</focalLength>
-		    <hackBaseline>0</hackBaseline>
-		  </plugin>
-		</sensor>
-	</gazebo>
   </xacro:macro>
 </robot>
